File: Spider.kicad_sch (KiCad schematic)
At the start: 47 parts

Commit message: split inputs and outputs, mounting holes, smd sockets
Parts:
- removed J1: (no value), symbol Connector_Generic:Conn_02x20_Odd_Even
- added H1, H2, H3, H4: (no value), symbol Mechanical:MountingHole
- added J1: Conn_02x12_Odd_Even, Connector_PinHeader_2.54mm:PinHeader_2x12_P2.54mm_Vertical_SMD, symbol Connector_Generic:Conn_02x12_Odd_Even
- added J2: Conn_02x08_Odd_Even, Connector_PinHeader_2.54mm:PinHeader_2x08_P2.54mm_Vertical_SMD, symbol Connector_Generic:Conn_02x08_Odd_Even
- C1, C2, C3, C4: value (none) -> 0.1uF; footprint (none) -> Capacitor_SMD:C_0603_1608Metric_Pad1.08x0.95mm_HandSolder
- D1, D2, D3, D4, D5, D6, D7, D8: value (none) -> z; footprint (none) -> LED_SMD:LED_0603_1608Metric_Pad1.05x0.95mm_HandSolder
- D9: value (none) -> ~; footprint (none) -> Diode_SMD:D_SMA
- J3: renamed from J2; value (none) -> USB_B_Micro; footprint (none) -> Connector_USB:USB_Micro-B_Amphenol_10103594-0001LF_Horizontal
- LOGO2: value (none) -> Logo OpenHW; footprint (none) -> Symbol:OSHW-Logo_7.5x8mm_SilkScreen
- LOGO3: value (none) -> Logo Spider; footprint (none) -> spider:spider_logo
- R1, R17, R2, R3, R4, R5, R6, R7, R8: value (none) -> 3.3K; footprint (none) -> Resistor_SMD:R_0805_2012Metric_Pad1.20x1.40mm_HandSolder
- R10, R11, R12, R13, R14, R15, R16, R9: value (none) -> 1K; footprint (none) -> Resistor_SMD:R_0805_2012Metric_Pad1.20x1.40mm_HandSolder
- SW1, SW2, SW3, SW4, SW5, SW6, SW7, SW8: value (none) -> SW_DPDT_x2; footprint (none) -> spider:SW_DPDT
- SW9: value (none) -> SW_Push_DPDT; footprint (none) -> spider:TL2230OAF140
- U1, U2: value (none) -> CD4050; footprint (none) -> Package_SO:SOIC-16W_7.5x10.3mm_P1.27mm
- U3: value (none) -> 74LS14; footprint (none) -> Package_SO:SSOP-14_5.3x6.2mm_P0.65mm
Connections:
- net GND: now also J1.23 (Pin_23), J1.24 (Pin_24)
- net LED1: now also J2.1 (Pin_1), J2.2 (Pin_2)
- net LED2: now also J2.3 (Pin_3), J2.4 (Pin_4)
- net LED3: now also J2.5 (Pin_5), J2.6 (Pin_6)
- net LED4: now also J2.7 (Pin_7), J2.8 (Pin_8)
- net LED5: now also J2.10 (Pin_10), J2.9 (Pin_9)
- net LED6: now also J2.11 (Pin_11), J2.12 (Pin_12)
- net LED7: now also J2.13 (Pin_13), J2.14 (Pin_14)
- net LED8: now also J2.15 (Pin_15), J2.16 (Pin_16)
- net PB1: now also J1.19 (Pin_19), J1.20 (Pin_20)
- net SW1: now also J1.3 (Pin_3), J1.4 (Pin_4)
- net SW2: now also J1.5 (Pin_5), J1.6 (Pin_6)
- net SW3: now also J1.7 (Pin_7), J1.8 (Pin_8)
- net SW4: now also J1.10 (Pin_10), J1.9 (Pin_9)
- net SW5: now also J1.11 (Pin_11), J1.12 (Pin_12)
- net SW6: now also J1.13 (Pin_13), J1.14 (Pin_14)
- net SW7: now also J1.15 (Pin_15), J1.16 (Pin_16)
- net SW8: now also J1.17 (Pin_17), J1.18 (Pin_18)
- net VCC: now also J1.1 (Pin_1), J1.2 (Pin_2)
- net nPB1: now also J1.21 (Pin_21), J1.22 (Pin_22)
Other:
- moved on the sheet: D9, J3, LOGO1, LOGO2, LOGO3
